Commit message: changed camera pose

File: src/mycobot_ros2/mycobot_description/urdf/sensors/intel_rgbd_cam_d435.urdf.xacro (robot description, xacro)
@@ -12,5 +12,5 @@
     <xacro:property name="d435_cam_depth_to_infra2_offset" value="-0.050"/>
     <xacro:property name="d435_cam_depth_to_color_offset" value="0.015"/>
-    <xacro:property name="camera_tilt_angle_deg" value="25"/>
+    <xacro:property name="camera_tilt_angle_deg" value="55"/>
     <link name="torso_link">
       <inertial>
@@ -53,10 +53,10 @@
       <parent link="$(arg prefix)base_link"/>
       <child link="torso_link"/>
-      <origin xyz="0.22 -0.30 0" rpy="0 0 0"/>
+      <origin xyz="0 0.40 0" rpy="0 0 0"/>
     </joint>
     <joint name="camera_head_joint" type="fixed">
       <parent link="torso_link"/>
       <child link="camera_head_link" />
-      <origin xyz="0 0.01 0.50" rpy="0.0 ${camera_tilt_angle_deg * M_PI / 180} ${M_PI/2}"/>
+      <origin xyz="0 -0.01 0.350" rpy="0.0 ${camera_tilt_angle_deg * M_PI / 180} ${-M_PI/2}"/>
     </joint>
     <link name="camera_head_link">

Commit message: changed camera and cube pose

File: src/mycobot_ros2/mycobot_description/urdf/sensors/intel_rgbd_cam_d435.urdf.xacro (robot description, xacro)
@@ -34,5 +34,5 @@
         </material>
         <geometry>
-          <box size="0.15 0.10 0.06" />
+          <box size="0.10 0.05 0.05" />
         </geometry>
       </visual>
@@ -53,5 +53,5 @@
       <parent link="$(arg prefix)base_link"/>
       <child link="torso_link"/>
-      <origin xyz="0 0.40 0" rpy="0 0 0"/>
+      <origin xyz="0 0.4 0" rpy="0 0 0"/>
     </joint>
     <joint name="camera_head_joint" type="fixed">

Commit message: Updated codebase with realtime inference and better auto data collection (excluding large files)

File: src/mycobot_ros2/mycobot_description/urdf/sensors/intel_rgbd_cam_d435.urdf.xacro (robot description, xacro)
@@ -12,5 +12,5 @@
     <xacro:property name="d435_cam_depth_to_infra2_offset" value="-0.050"/>
     <xacro:property name="d435_cam_depth_to_color_offset" value="0.015"/>
-    <xacro:property name="camera_tilt_angle_deg" value="55"/>
+    <xacro:property name="camera_tilt_angle_deg" value="25"/>
     <link name="torso_link">
       <inertial>
@@ -53,10 +53,10 @@
       <parent link="$(arg prefix)base_link"/>
       <child link="torso_link"/>
-      <origin xyz="0 0.4 0" rpy="0 0 0"/>
+      <origin xyz="0 0.48 0" rpy="0 0 0"/>
     </joint>
     <joint name="camera_head_joint" type="fixed">
       <parent link="torso_link"/>
       <child link="camera_head_link" />
-      <origin xyz="0 -0.01 0.350" rpy="0.0 ${camera_tilt_angle_deg * M_PI / 180} ${-M_PI/2}"/>
+      <origin xyz="0 -0.01 0.250" rpy="0.0 ${camera_tilt_angle_deg * M_PI / 180} ${-M_PI/2}"/>
     </joint>
     <link name="camera_head_link">
@@ -135,6 +135,6 @@
           <horizontal_fov>1.5184</horizontal_fov>
           <image>
-            <width>424</width>
-            <height>240</height>
+            <width>640</width>
+            <height>480</height>
           </image>
           <clip>
